File: kicad/usb-c.kicad_sch (KiCad schematic)
At the start: 8 parts, among them J201 USB_C_Receptacle_USB2.0_16P

Commit message: add some assembly files, but transition towards all hand
Parts:
- D201: footprint Package_SON:Texas_DPY0002A_0.6x1mm_P0.65mm -> Diode_SMD:D_SOD-523; JLC (none) -> XXXXXX; LCSC (none) -> XXXXXX
- D202, D203, J201, TP201, TP202: JLC (none) -> XXXXXX; LCSC (none) -> XXXXXX
- R204, R205: JLC (none) -> 0603
Changed lines of the file:
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@@
 			)
 		)
-		(property "Footprint" "Package_SON:Texas_DPY0002A_0.6x1mm_P0.65mm"
+		(property "Footprint" "Diode_SMD:D_SOD-523"
 			(at 113.03 91.44 0)
 			(effects
@@
 		)
 		(property "Description" "Zener diode"
+			(at 113.03 91.44 0)
+			(effects
+				(font
+					(size 1.27 1.27)
+				)
+				(hide yes)
+			)
+		)
+		(property "JLC" "XXXXXX"
+			(at 113.03 91.44 0)
+			(effects
+				(font
+					(size 1.27 1.27)
+				)
+				(hide yes)
+			)
+		)
+		(property "LCSC" "XXXXXX"
 			(at 113.03 91.44 0)
 			(effects
@@
 			)
 		)
+		(property "JLC" "XXXXXX"
+			(at 133.35 140.97 0)
+			(effects
+				(font
+					(size 1.27 1.27)
+				)
+				(hide yes)
+			)
+		)
+		(property "LCSC" "XXXXXX"
+			(at 133.35 140.97 0)
+			(effects
+				(font
+					(size 1.27 1.27)
+				)
+				(hide yes)
+			)
+		)
 		(pin "1"
 		)
@@
 			)
 		)
+		(property "JLC" "0603"
+			(at 140.97 106.68 0)
+			(effects
+				(font
+					(size 1.27 1.27)
+				)
+				(hide yes)
+			)
+		)
 		(pin "1"
 		)
@@
 			)
 		)
+		(property "JLC" "XXXXXX"
+			(at 120.65 110.49 0)
+			(effects
+				(font
+					(size 1.27 1.27)
+				)
+				(hide yes)
+			)
+		)
+		(property "LCSC" "XXXXXX"
+			(at 120.65 110.49 0)
+			(effects
+				(font
+					(size 1.27 1.27)
+				)
+				(hide yes)
+			)
+		)
 		(pin "1"
 		)
@@
 			)
 		)
+		(property "JLC" "XXXXXX"
+			(at 133.35 135.89 0)
+			(effects
+				(font
+					(size 1.27 1.27)
+				)
+				(hide yes)
+			)
+		)
+		(property "LCSC" "XXXXXX"
+			(at 133.35 135.89 0)
+			(effects
+				(font
+					(size 1.27 1.27)
+				)
+				(hide yes)
+			)
+		)
 		(pin "1"
 		)
@@
 		)
 		(property "Description" "Zener diode"
+			(at 115.57 118.11 0)
+			(effects
+				(font
+					(size 1.27 1.27)
+				)
+				(hide yes)
+			)
+		)
+		(property "JLC" "XXXXXX"
+			(at 115.57 118.11 0)
+			(effects
+				(font
+					(size 1.27 1.27)
+				)
+				(hide yes)
+			)
+		)
+		(property "LCSC" "XXXXXX"
 			(at 115.57 118.11 0)
 			(effects
@@
 			)
 		)
+		(property "JLC" "XXXXXX"
+			(at 92.71 109.22 0)
+			(effects
+				(font
+					(size 1.27 1.27)
+				)
+				(hide yes)
+			)
+		)
+		(property "LCSC" "XXXXXX"
+			(at 92.71 109.22 0)
+			(effects
+				(font
+					(size 1.27 1.27)
+				)
+				(hide yes)
+			)
+		)
 		(pin "A4"
 		)
@@
 			(at 132.08 106.68 0)
 			(effects
+				(font
+					(size 1.27 1.27)
+				)
+				(hide yes)
+			)
+		)
+		(property "JLC" "0603"
+			(at 132.08 106.68 0)
+			(effects

Commit message: new battery management w/ separate LDO/charger almost done
Other:
- company: Author: Lucas Merritt -> Mosaic Labs
Changed lines of the file:
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@@
 		(date "2024-09-02")
 		(rev "1")
-		(company "Author: Lucas Merritt")
+		(company "Mosaic Labs")
+		(comment 1 "Lucas Merritt")
 	)
 	(junction

Commit message: finish management schematic, ready for PCB
Parts:
- TP201: value CC1_TP -> CC1_TEST
- TP202: value CC2_TP -> CC2_TEST
Changed lines of the file:
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@@
 			)
 		)
-		(property "Value" "CC2_TP"
+		(property "Value" "CC2_TEST"
 			(at 138.43 142.2399 90)
 			(effects
@@
 			)
 		)
-		(property "Value" "CC1_TP"
+		(property "Value" "CC1_TEST"
 			(at 138.43 137.1599 90)
 			(effects

Commit message: finish battery PCB layout, PCB refactoring
Parts:
- renumbered R204 to R201, R205 to R202
Changed lines of the file:
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@@
 		(dnp no)
 		(fields_autoplaced yes)
-		(property "Reference" "R205"
+		(property "Reference" "R202"
 			(at 143.51 105.4099 0)
 			(effects
@@
 			(project "kicad"
 				(path "/97e37379-fec6-4f0d-82d9-4ea53516bb02/32d68f15-4a24-4df9-a303-ad9032613b76"
-					(reference "R205")
+					(reference "R202")
 					(unit 1)
 				)
@@
 		(dnp no)
 		(fields_autoplaced yes)
-		(property "Reference" "#PWR0208"
+		(property "Reference" "#PWR0205"
 			(at 140.97 116.84 0)
 			(effects
@@
 			(project "kicad"
 				(path "/97e37379-fec6-4f0d-82d9-4ea53516bb02/32d68f15-4a24-4df9-a303-ad9032613b76"
-					(reference "#PWR0208")
+					(reference "#PWR0205")
 					(unit 1)
 				)
@@
 		(on_board yes)
 		(dnp no)
-		(property "Reference" "R204"
+		(property "Reference" "R201"
 			(at 133.858 105.41 0)
 			(effects
@@
 			(project "kicad"
 				(path "/97e37379-fec6-4f0d-82d9-4ea53516bb02/32d68f15-4a24-4df9-a303-ad9032613b76"
-					(reference "R204")
-					(unit 1)
-				)
+					(reference "R201")
+					(unit 1)
+				)

Commit message: Microcontroller additions
Parts:
- removed TP201: CC1_TEST, TestPoint:TestPoint_Pad_D1.5mm, symbol Connector:TestPoint
- removed TP202: CC2_TEST, TestPoint:TestPoint_Pad_D1.5mm, symbol Connector:TestPoint
Changed lines of the file:
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@@
 		(company "Mosaic Labs")
 		(comment 1 "Lucas Merritt")
+		(comment 2 "Rev. 1 verified")
+		(comment 3 "Final ready")
 	)
 	(junction
@@
 	(wire
 		(pts
-			(xy 133.35 140.97) (xy 125.73 140.97)
-		)
-		(stroke
-			(width 0)
-			(type default)
-		)
-	)
-	(wire
-		(pts
 			(xy 107.95 87.63) (xy 113.03 87.63)
 		)
@@
 		(pts
 			(xy 140.97 99.06) (xy 140.97 102.87)
-		)
-		(stroke
-			(width 0)
-			(type default)
-		)
-	)
-	(wire
-		(pts
-			(xy 133.35 135.89) (xy 125.73 135.89)
 		)
 		(stroke
@@
 			)
 			(justify right bottom)
-		)
-	)
-	(label "CC2_T"
-		(at 125.73 140.97 0)
-		(fields_autoplaced yes)
-		(effects
-			(font
-				(size 1.27 1.27)
-			)
-			(justify left bottom)
-		)
-	)
-	(label "CC1_T"
-		(at 125.73 135.89 0)
-		(fields_autoplaced yes)
-		(effects
-			(font
-				(size 1.27 1.27)
-			)
-			(justify left bottom)
 		)
 	)
@@
 	)
 	(symbol
-		(lib_id "Connector:TestPoint")
-		(at 133.35 140.97 270)
-		(unit 1)
-		(exclude_from_sim no)
-		(in_bom yes)
-		(on_board yes)
-		(dnp no)
-		(fields_autoplaced yes)
-		(property "Reference" "TP202"
-			(at 138.43 139.6999 90)
-			(effects
-				(font
-					(size 1.27 1.27)
-				)
-				(justify left)
-			)
-		)
-		(property "Value" "CC2_TEST"
-			(at 138.43 142.2399 90)
-			(effects
-				(font
-					(size 1.27 1.27)
-				)
-				(justify left)
-			)
-		)
-		(property "Footprint" "TestPoint:TestPoint_Pad_D1.5mm"
-			(at 133.35 146.05 0)
-			(effects
-				(font
-					(size 1.27 1.27)
-				)
-				(hide yes)
-			)
-		)
-		(property "Datasheet" "~"
-			(at 133.35 146.05 0)
-			(effects
-				(font
-					(size 1.27 1.27)
-				)
-				(hide yes)
-			)
-		)
-		(property "Description" "test point"
-			(at 133.35 140.97 0)
-			(effects
-				(font
-					(size 1.27 1.27)
-				)
-				(hide yes)
-			)
-		)
-		(property "JLC" "XXXXXX"
-			(at 133.35 140.97 0)
-			(effects
-				(font
-					(size 1.27 1.27)
-				)
-				(hide yes)
-			)
-		)
-		(property "LCSC" "XXXXXX"
-			(at 133.35 140.97 0)
-			(effects
-				(font
-					(size 1.27 1.27)
-				)
-				(hide yes)
-			)
-		)
-		(pin "1"
-		)
-		(instances
-			(project "kicad"
-				(path "/97e37379-fec6-4f0d-82d9-4ea53516bb02/32d68f15-4a24-4df9-a303-ad9032613b76"
-					(reference "TP202")
-					(unit 1)
-				)
-			)
-		)
-	)
-	(symbol
 		(lib_id "Device:R")
 		(at 140.97 106.68 0)
@@
 					(unit 1)
 				)
-			)
-		)
-	)
-	(symbol
-		(lib_id "Connector:TestPoint")
-		(at 133.35 135.89 270)
-		(unit 1)
-		(exclude_from_sim no)
-		(in_bom yes)
-		(on_board yes)
-		(dnp no)
-		(fields_autoplaced yes)
-		(property "Reference" "TP201"
-			(at 138.43 134.6199 90)
-			(effects
-				(font
-					(size 1.27 1.27)
-				)
-				(justify left)
-			)
-		)
-		(property "Value" "CC1_TEST"
-			(at 138.43 137.1599 90)
-			(effects
-				(font
-					(size 1.27 1.27)
-				)
-				(justify left)
-			)
-		)
-		(property "Footprint" "TestPoint:TestPoint_Pad_D1.5mm"
-			(at 133.35 140.97 0)
-			(effects
-				(font
-					(size 1.27 1.27)
-				)
-				(hide yes)
-			)
-		)
-		(property "Datasheet" "~"
-			(at 133.35 140.97 0)
-			(effects
-				(font
-					(size 1.27 1.27)
-				)
-				(hide yes)
-			)
-		)
-		(property "Description" "test point"
-			(at 133.35 135.89 0)
-			(effects
-				(font
-					(size 1.27 1.27)
-				)
-				(hide yes)
-			)
-		)
-		(property "JLC" "XXXXXX"
-			(at 133.35 135.89 0)
-			(effects
-				(font
-					(size 1.27 1.27)
-				)
-				(hide yes)
-			)
-		)
-		(property "LCSC" "XXXXXX"
-			(at 133.35 135.89 0)
-			(effects
-				(font
-					(size 1.27 1.27)
-				)
-				(hide yes)
-			)
-		)
-		(pin "1"
-		)
-		(instances
-			(project "kicad"
-				(path "/97e37379-fec6-4f0d-82d9-4ea53516bb02/32d68f15-4a24-4df9-a303-ad9032613b76"
-					(reference "TP201")
-					(unit 1)
-				)

Commit message: Unfinished switch additions and fixes
Other:
- note added: "Make sure to place these diodes correctly"
- note added: "NC"
Changed lines of the file:
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@@
+		)
+	)
+	(text "NC"
+		(exclude_from_sim no)
+		(at 110.49 123.19 0)
+		(effects
+			(font
+				(size 1.27 1.27)
+			)
 		)
 	)
@@
 		(effects
 			(font
+				(size 1.27 1.27)
+			)
+		)
+	)
+	(text "Make sure to\nplace these\ndiodes correctly"
+		(exclude_from_sim no)
+		(at 120.396 129.032 0)
+		(effects
+			(font

Commit message: Small switch updates and fixes
Other:
- note added: "Or ESD441 if in stock"
Changed lines of the file:
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@@
+		)
+	)
+	(text "Or ESD441 if in stock"
+		(exclude_from_sim no)
+		(at 143.51 93.218 0)
+		(effects
+			(font
+				(size 1.27 1.27)
+			)
 		)
 	)

Commit message: Begin PCB, update footprints
Parts:
- R201, R202: footprint Resistor_SMD:R_0603_1608Metric_Pad0.98x0.95mm_HandSolder -> Resistor_SMD:R_0402_1005Metric
Changed lines of the file:
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@@
 			)
 		)
-		(property "Footprint" "Resistor_SMD:R_0603_1608Metric_Pad0.98x0.95mm_HandSolder"
+		(property "Footprint" "Resistor_SMD:R_0402_1005Metric"
 			(at 139.192 106.68 90)
 			(effects
@@
 			)
 		)
-		(property "Footprint" "Resistor_SMD:R_0603_1608Metric_Pad0.98x0.95mm_HandSolder"
+		(property "Footprint" "Resistor_SMD:R_0402_1005Metric"
 			(at 130.302 106.68 90)
 			(effects
