File: kicad/usb-c.kicad_sch (KiCad schematic)
At the start: 6 parts, among them J201 USB_C_Receptacle_USB2.0_16P

Commit message: Minor schematic fixes and PCB trace progress
Connections:
- net DM renamed D-
- net DP renamed D+
Changed lines of the file:
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@@
 		)
 	)
-	(hierarchical_label "DM"
-		(shape output)
+	(hierarchical_label "D-"
+		(shape bidirectional)
 		(at 120.65 106.68 90)
 		(fields_autoplaced yes)
@@
 		)
 	)
-	(hierarchical_label "DP"
-		(shape output)
+	(hierarchical_label "D+"
+		(shape bidirectional)
 		(at 115.57 114.3 90)
 		(fields_autoplaced yes)

Commit message: start v3, complete pcb restart and remove haptics
Parts:
- renumbered D203 to D202, D202 to D203
