File: kicad/microcontroller.kicad_sch (KiCad schematic)
At the start: 21 parts, among them Q701 DMG1012T, U701 MLPF-WB55-01E3, U702 STM32WB55RGVx, Y701 32M

Commit message: v2.0.2
Parts:
- removed Q701: DMG1012T, Package_TO_SOT_SMD:SOT-523, symbol Transistor_FET:DMG1012T
- removed R701: 100k, Resistor_SMD:R_0402_1005Metric, symbol Device:R
- removed R702: 10k, Resistor_SMD:R_0402_1005Metric, symbol Device:R
- added C714, C715: 10pF, Capacitor_SMD:C_0402_1005Metric, symbol Device:C
- added Y702: NX2012_32K768, Crystal:Crystal_SMD_2012-2Pin_2.0x1.2mm, symbol Device:Crystal
- Y701: value 32M -> 8Y-32.000MAAV-T
Connections:
- net BT1: now also U702.5 (PH3)
- net GND: now also C714.2, C715.2
- net at U702.3 (PC14): now also C714.1, Y702.1
- net at U702.4 (PC15): now also C715.1, Y702.2
Other:
- note added: "OSC32_IN"
- note added: "OSC32_OUT"
- note removed: "BT1 defaults high, so BOOT0 defaults low, changes when pressed"
- note removed: "If BT1 held on reset, trigger bootloader for USB DFU"

Commit message: start v3, complete pcb restart and remove haptics
Parts:
- renumbered AE701 to AE601, C705 to C601, C707 to C602, C710 to C603, C711 to C604, C703 to C605, C704 to C606, C706 to C607, C708 to C608, C709 to C609, C712 to C610, C713 to C611, C702 to C612, C701 to C613, C714 to C614, C715 to C615, L701 to L601, U701 to U601, U702 to U602, Y701 to Y601, Y702 to Y602
Connections:
- net I2C1_SCL: no longer names the net of U602.6 (PB8)
- net I2C1_SDA: no longer names the net of U602.7 (PB9)
- net LED_BATT: no longer names the net of U602.38 (PB0)
- net LED_F1: no longer names the net of U602.39 (PB1)
- net LED_F2: no longer names the net of U602.65 (PB5)
- net TIM2_CH1: no longer names the net of U602.15 (PA0)
